File: updatedCM5.kicad_pcb (KiCad board)
At the start: 4 copper layers, 160 x 90 mm, 61 parts, among them J11 USB_C_Receptacle_USB2.0, J14 JST_SHBM04B-SRSS-TB, J3 Conn_01x03, J4 Bus_M.2_Socket_M, J5 Conn_01x22_Female, J6 THD-02-R, J7 Micro_SD_Card_Det, J8 THD-20-R, SW1 Right angle Tact button, U18 RT9742GGJ5, U6 AP22653W6, U7 ASEK-32.768KHZ-L-R-T, U8 AP3441SHE-7B

Commit message: end of jan 11th
Parts:
- removed H1: MountingHole, CM5IO:MountingHole_2.7mm_M2.5_DIN965
- added J2: Conn_02x07_Odd_Even, Connector_PinHeader_2.54mm:PinHeader_2x07_P2.54mm_Vertical, F.Cu at (83.9, 96.0)
- moved Module1 115.4 mm to (88.5, 116.7), turned to -90 degrees
- moved J7 115.4 mm to (86.6, 138.1), turned to 90 degrees
Connections:
- C2 pad 1: /CM5_HighSpeed/+5v -> /+5v
- Module1 pad 101: /CM5_HighSpeed/USBOTG_ID -> /CM5_GPIO ( Ethernet, GPIO, SDCARD)/USBOTG
- U6 pad 1: /CM5_HighSpeed/+5v -> /+5v
Routing:
- net GND: track 764.8 -> 1121.9 mm, vias 476 -> 474
- net /CM5_HighSpeed/DPHY1_C_N: track 66.1 -> 360.6 mm, vias 2 -> 6
- net /CM5_HighSpeed/HDMI0_HOTPLUG: track 102.3 -> 0.00 mm, vias 2 -> 0
- net /CM5_HighSpeed/HDMI0_SDA: track 100.2 -> 0.00 mm, vias 2 -> 0
- net /CM5_HighSpeed/HDMI0_CEC: track 95.9 -> 0.00 mm, vias 2 -> 0
- net /CM5_HighSpeed/DPHY1_D0_P: track 67.7 -> 162.9 mm
- net /CM5_HighSpeed/HDMI0_SCL: track 95.2 -> 0.90 mm, vias 0 -> 1
- net /CM5_HighSpeed/DPHY1_D1_P: track 66.3 -> 160.2 mm, vias 2 -> 3
- net /CM5_HighSpeed/HDMI0_CK_N: track 93.5 -> 0.00 mm
- net /CM5_HighSpeed/DPHY1_D2_P: track 66.7 -> 160.2 mm
- net /CM5_HighSpeed/USB3-1-D_N: track 75.0 -> 168.5 mm
- net /CM5_HighSpeed/HDMI0_CK_P: track 93.5 -> 0.00 mm
- net /CM5_HighSpeed/HDMI0_D0_N: track 92.0 -> 0.00 mm
- net /CM5_HighSpeed/HDMI0_D0_P: track 91.9 -> 0.00 mm
- net /CM5_HighSpeed/HDMI0_D1_N: track 90.4 -> 0.00 mm
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